File: tut_instructables.kicad_sch (KiCad schematic)
At the start: 31 parts, among them J1 USB4110GFA, J2 Conn_01x08_Pin, SW1 CK_KMS2xxGP, SW2 CK_KMS2xxGP, U1 AMS1117-3.3, U2 ESP32-C3-WROOM-02

Commit message: added all the footprints
Parts:
- D1: footprint Diode_THT:D_DO-41_SOD81_P10.16mm_Horizontal -> Diode_SMD:D_0201_0603Metric
- J2: footprint (none) -> Connector_PinHeader_2.00mm:PinHeader_1x08_P2.00mm_Vertical
Changed lines of the file:
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@@
 			)
 		)
-		(property "Footprint" "Diode_THT:D_DO-41_SOD81_P10.16mm_Horizontal"
+		(property "Footprint" "Diode_SMD:D_0201_0603Metric"
 			(at 91.44 26.035 0)
 			(effects
@@
 			)
 		)
-		(property "Footprint" ""
+		(property "Footprint" "Connector_PinHeader_2.00mm:PinHeader_1x08_P2.00mm_Vertical"
 			(at 120.65 158.75 0)
 			(effects
